File: contrib/bmp22/bmp22/target_interface.sch (KiCad schematic (older format))
At the start: 30 parts, among them J201 Conn_01x10_Male, J203 PH1x4, Q201 DMG1023UV-7, Q202 DMG1024UV-7, Q203 DMG1024UV-7, U201 SN74LVC2T45DCUR, U202 SN74LVC2T45DCUR, U203 SN74LVC2T45DCUR, U204 SN74LVC2T45DCUR

Commit message: added footprints
Parts:
- C201, C202, C203, C204, C205, C206, C207, C208: footprint (none) -> Capacitor_SMD:C_0402_1005Metric
- J201: footprint (none) -> Connector_PinHeader_1.27mm:PinHeader_2x05_P1.27mm_Vertical_SMD
- J202: renamed from J203; footprint (none) -> Connector_JST:JST_PH_S4B-PH-SM4-TB_1x04-1MP_P2.00mm_Horizontal
- JP201, JP202, R201, R202, R203, R204, R205, R206, R207, R208, R209, R210, R211: footprint (none) -> Resistor_SMD:R_0402_1005Metric
- Q201, Q202, Q203: footprint (none) -> Package_TO_SOT_SMD:SOT-563

Commit message: created layout
Parts:
- removed Q202: DMG1024UV-7, Package_TO_SOT_SMD:SOT-563, symbol Device:Q_DUAL_PMOS_S1G1D2S2G2D1
- added unit 2 of Q201
Connections:
- net PWR_BR: now also Q201.5 (G)
- net TPWR: now also Q201.3 (D)
- net xRXD: now also R209.2; no longer R208.2
- net xTXD: now also R208.2; no longer R209.2
- net at Q201.1 (S), R210.1: now also Q201.4 (S)
Changed lines of the file:
@@
 	1    0    0    -1
 $EndComp
+Text GLabel 7700 3150 0    50   Input ~ 0
+xRXD
 Text GLabel 7700 2950 0    50   Input ~ 0
-xRXD
-Text GLabel 7700 3150 0    50   Input ~ 0
 xTXD
 Text GLabel 3550 1900 2    50   Input ~ 0
@@
 	0    -1   -1   0
 $EndComp
-$Comp
-L Device:Q_DUAL_PMOS_S1G1D2S2G2D1 Q201
-U 1 1 5F22768C
-P 6100 3400
-F 0 "Q201" H 6350 3450 50  0000 C CNN
-F 1 "DMG1023UV-7" V 5800 3400 50  0000 C CNN
-F 2 "Package_TO_SOT_SMD:SOT-563" H 6150 3400 50  0001 C CNN
-F 3 "~" H 6150 3400 50  0001 C CNN
-	1    6100 3400
-	0    1    1    0
-$EndComp
-$Comp
-L Device:Q_DUAL_PMOS_S1G1D2S2G2D1 Q202
-U 1 1 5F227692
-P 6100 4100
-F 0 "Q202" H 6350 4150 50  0000 C CNN
-F 1 "DMG1024UV-7" V 5800 4100 50  0000 C CNN
-F 2 "Package_TO_SOT_SMD:SOT-563" H 6150 4100 50  0001 C CNN
-F 3 "~" H 6150 4100 50  0001 C CNN
-	1    6100 4100
-	0    1    -1   0
-$EndComp
 Wire Wire Line
 	6100 3200 5550 3200
@@
 Wire Wire Line
 	8400 1000 8400 1150
+$Comp
+L Device:Q_DUAL_PMOS_S1G1D2S2G2D1 Q201
+U 1 1 5F22768C
+P 6100 3400
+F 0 "Q201" V 6250 3700 50  0000 C CNN
+F 1 "DMG1023UV-7" V 5800 3400 50  0000 C CNN
+F 2 "Package_TO_SOT_SMD:SOT-563" H 6150 3400 50  0001 C CNN
+F 3 "~" H 6150 3400 50  0001 C CNN
+	1    6100 3400
+	0    1    1    0
+$EndComp
+$Comp
+L Device:Q_DUAL_PMOS_S1G1D2S2G2D1 Q201
+U 2 1 5F16690A
+P 6100 4100
+F 0 "Q201" V 6250 4400 50  0000 C CNN
+F 1 "DMG1023UV-7" V 5800 4100 50  0000 C CNN
+F 2 "Package_TO_SOT_SMD:SOT-563" H 6150 4100 50  0001 C CNN
+F 3 "~" H 6150 4100 50  0001 C CNN
+	2    6100 4100
+	0    1    -1   0
+$EndComp
 $EndSCHEMATC
